File: Hardware/Citcuito.sch (KiCad schematic (older format))
At the start: 56 parts, among them J1 ESP32 DEV KIT V1

Commit message: Sla kk
Parts:
- gave numbers to parts that had none: 55
- renumbered J1 to J3
Other:
- note added: "Buzzer controlado por frequencia"
- note added: "Controle de leds RGB com PWM"
- note added: "Matriz de botões 3x3"
- note added: "Modulos conectados por headers"
- note added: "Saídas digitais com led"
- note added: "Sensor de luminosidade e infravermelho para proximidade ambos com buffer"
